File: pcb/nikon.kicad_pcb (KiCad board)
At the start: 2 copper layers, 143.3 x 125.7 mm, 83 parts, among them J1 USB_C_Receptacle_USB2.0, J2 AVR-ISP-6, SW1 SW_Push, U1 ATmega32U4-AU, Y1 16MHz

Commit message: ...
Parts:
- added C4: 4.7u, Capacitor_SMD:C_0805_2012Metric_Pad1.18x1.45mm_HandSolder, B.Cu at (134.0, 95.4)
- added C5: 0.1u, Capacitor_SMD:C_0805_2012Metric_Pad1.18x1.45mm_HandSolder, B.Cu at (139.9, 100.3)
- added C6: 0.1u, Capacitor_SMD:C_0805_2012Metric_Pad1.18x1.45mm_HandSolder, B.Cu at (128.6, 121.9)
- added C7: 0.1u, Capacitor_SMD:C_0805_2012Metric_Pad1.18x1.45mm_HandSolder, B.Cu at (123.0, 108.0)
- added C8: 0.1u, Capacitor_SMD:C_0805_2012Metric_Pad1.18x1.45mm_HandSolder, B.Cu at (123.0, 100.7)
- added J3: SJ2-35043A-SMT-TR, nikon:CUI_SJ2-35043A-SMT-TR, B.Cu at (158.7, 90.4)
- moved R6 63.1 mm to (124.7, 112.1), turned to 180 degrees
- moved R4 58.9 mm to (143.0, 36.4), turned to 90 degrees
- moved R2 55.4 mm to (146.3, 35.2)
- moved R5 53.1 mm to (140.5, 36.4), turned to 90 degrees
- moved F1 52.7 mm to (137.2, 36.4), turned to -90 degrees
- moved R3 51.5 mm to (146.3, 37.6)
- moved R1 49.3 mm to (149.6, 36.4), turned to -90 degrees
- moved C1 40.1 mm to (138.4, 95.4)
- moved D33 10.9 mm to (151.2, 121.1)
- moved C3 10.3 mm to (143.2, 97.9), turned to 180 degrees
- moved Y1 6.97 mm to (143.2, 104.1), turned to 90 degrees
- moved C2 5.22 mm to (139.9, 106.9), turned to 90 degrees
- moved U1 2.19 mm to (131.4, 103.7), turned to -90 degrees
- moved J1 0.50 mm to (143.2, 25.2)
- renumbered R2 to R1, R5 to R2, R6 to R3, R3 to R4, R4 to R5, R1 to R6
Connections:
- J1 pad A8: Net-(J1-PadA8) -> unconnected-(J1-PadA8)
- J1 pad B8: Net-(J1-PadB8) -> unconnected-(J1-PadB8)
- U1 pad 1: Net-(U1-Pad1) -> unconnected-(U1-Pad1)
- U1 pad 12: Net-(U1-Pad12) -> unconnected-(U1-Pad12)
- U1 pad 18: Net-(U1-Pad18) -> unconnected-(U1-Pad18)
- U1 pad 19: Net-(U1-Pad19) -> unconnected-(U1-Pad19)
- U1 pad 20: Net-(U1-Pad20) -> unconnected-(U1-Pad20)
- U1 pad 21: Net-(U1-Pad21) -> unconnected-(U1-Pad21)
- U1 pad 22: Net-(U1-Pad22) -> unconnected-(U1-Pad22)
- U1 pad 25: Net-(U1-Pad25) -> unconnected-(U1-Pad25)
- U1 pad 26: Net-(U1-Pad26) -> unconnected-(U1-Pad26)
- U1 pad 27: Net-(U1-Pad27) -> unconnected-(U1-Pad27)
- U1 pad 28: Net-(U1-Pad28) -> unconnected-(U1-Pad28)
- U1 pad 29: Net-(U1-Pad29) -> unconnected-(U1-Pad29)
- U1 pad 30: Net-(U1-Pad30) -> unconnected-(U1-Pad30)
- U1 pad 31: Net-(U1-Pad31) -> unconnected-(U1-Pad31)
- U1 pad 32: Net-(U1-Pad32) -> unconnected-(U1-Pad32)
- U1 pad 36: Net-(U1-Pad36) -> unconnected-(U1-Pad36)
- U1 pad 37: Net-(U1-Pad37) -> unconnected-(U1-Pad37)
- U1 pad 38: Net-(U1-Pad38) -> unconnected-(U1-Pad38)
- U1 pad 39: Net-(U1-Pad39) -> unconnected-(U1-Pad39)
- U1 pad 40: Net-(U1-Pad40) -> unconnected-(U1-Pad40)
- U1 pad 41: Net-(U1-Pad41) -> unconnected-(U1-Pad41)
- U1 pad 42: Net-(U1-Pad42) -> unconnected-(U1-Pad42)
- U1 pad 8: Net-(U1-Pad8) -> unconnected-(U1-Pad8)
Routing:
- net /D-: track 0.00 -> 70.8 mm
- net /D+: track 0.00 -> 68.2 mm
- net GND: track 0.00 -> 15.9 mm
- net /USB_D+: track 0.00 -> 10.4 mm
- net /USB_D-: track 0.00 -> 7.61 mm
Other:
- board size 143.3 x 125.7 mm -> 143.3 x 124.7 mm
- net class Default removed

Commit message: update
Parts:
- moved J3 31.2 mm to (147.8, 61.2)
- moved C3 18.4 mm to (137.5, 115.4), turned to 90 degrees
- moved Y1 16.4 mm to (131.3, 115.4), turned to 0 degrees
- moved R6 15.1 mm to (123.3, 97.1), turned to 90 degrees
- moved C1 14.4 mm to (140.1, 109.6), turned to -90 degrees
- moved C7 13.4 mm to (127.5, 95.3), turned to 0 degrees
- moved C8 12.9 mm to (134.7, 95.3), turned to 180 degrees
- moved C5 12.9 mm to (135.1, 112.2), turned to 180 degrees
- moved C2 12.6 mm to (128.5, 112.2), turned to 0 degrees
- moved C4 10.4 mm to (140.1, 103.7), turned to 90 degrees
- moved U1 0.27 mm to (131.7, 103.8), turned to 180 degrees
Routing:
- net +5V: track 0.00 -> 12.7 mm
- net GND: track 15.9 -> 27.8 mm
- net /XTAL1: track 0.00 -> 11.7 mm
- net /XTAL2: track 0.00 -> 10.4 mm
- net Net-(C1-Pad1): track 0.00 -> 9.67 mm
- net /D+: track 68.2 -> 69.7 mm
Other:
- outline, holes or cut-outs redrawn
