File: pcb-left/nikon.kicad_sch (KiCad schematic)
At the start: 89 parts, among them J1 USB_C_Receptacle_USB2.0, J2 AVR-ISP-6, J3 SJ2-35043A-SMT-TR, SW1 SW_Push, U1 ATmega32U4-AU, Y1 16MHz

Commit message: both halves
Parts:
- removed J3: SJ2-35043A-SMT-TR, nikon:CUI_SJ2-35043A-SMT-TR, symbol nikon:SJ2-35043A-SMT-TR
- added J3: SJ2-35894A-SMT-TR, CUI_SJ2-35894A-SMT-TR, symbol nikon:SJ2-35894A-SMT-TR
- added R? (x2): R, symbol Device:R
Connections:
- net +5V: now also J3.4, R?.1, R?.1
- net GND: now also J3.1
- net SCL: now reaches U1.18 (PD0)
- net SCL: now also J3.2, R?.2
- net SDA: now reaches U1.19 (PD1)
- net SDA: now also J3.3, R?.2
