File: pcb-right/nikon.kicad_pcb (KiCad board)
At the start: 2 copper layers, 143.3 x 124.7 mm, 89 parts, among them J1 USB_C_Receptacle_USB2.0, J2 AVR-ISP-6, J3 SJ2-35043A-SMT-TR, SW1 SW_Push, U1 ATmega32U4-AU, Y1 16MHz

Commit message: both halves
Parts:
- moved SW1 127.2 mm to (225.7, 91.7), turned to 180 degrees
- moved J3 78.0 mm to (225.5, 68.7)
- moved C3 77.6 mm to (214.8, 122.9)
- moved C5 77.6 mm to (212.4, 119.7)
- moved C6 77.6 mm to (205.9, 129.4)
- moved D25 77.6 mm to (195.5, 134.8)
- moved D30 77.6 mm to (210.2, 143.4)
- moved D33 77.6 mm to (228.5, 128.6)
- moved D34 77.6 mm to (225.0, 151.9)
- moved MX33 77.6 mm to (228.3, 118.1)
- moved D1 77.6 mm to (105.2, 48.7)
- moved D10 77.6 mm to (122.0, 116.7)
- moved D11 77.6 mm to (140.0, 48.7)
- moved D12 77.6 mm to (140.0, 65.7)
- moved D13 77.6 mm to (140.0, 82.7)
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Routing:
- net Net-(J1-PadB5): track 0.00 -> 16.2 mm, vias 0 -> 1
- net +5V: track 12.7 -> 27.0 mm, vias 0 -> 2
- net Net-(F1-Pad2): track 0.00 -> 5.77 mm
- net Net-(D34-Pad2): track 0.00 -> 5.27 mm
- net Net-(D30-Pad2): track 0.00 -> 5.26 mm
- net Net-(D25-Pad2): track 0.00 -> 5.25 mm
- net Net-(J1-PadA5): track 0.00 -> 4.50 mm
- net Net-(D9-Pad2): track 0.00 -> 4.13 mm
- net Net-(D8-Pad2): track 0.00 -> 4.13 mm
- net Net-(D7-Pad2): track 0.00 -> 4.13 mm
- net Net-(D6-Pad2): track 0.00 -> 4.13 mm
- net Net-(D29-Pad2): track 0.00 -> 4.13 mm
- net Net-(D28-Pad2): track 0.00 -> 4.13 mm
- net Net-(D27-Pad2): track 0.00 -> 4.13 mm
- net Net-(D26-Pad2): track 0.00 -> 4.13 mm
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Other:
- outline, holes or cut-outs redrawn
